Commit message: Change axis 1 and 4 limits

File: fanuc_m10ia_support/urdf/m10ia_macro.xacro (robot description, xacro)
@@ -117,5 +117,5 @@
       <child link="${prefix}link_1"/>
       <axis xyz="0 0 1"/>
-      <limit lower="-3.14" upper="3.14" effort="0" velocity="3.67"/>
+      <limit lower="-0.78" upper="0.78" effort="0" velocity="3.67"/>
     </joint>
     <joint name="${prefix}joint_2" type="revolute">
@@ -138,5 +138,5 @@
       <child link="${prefix}link_4"/>
       <axis xyz="-1 0 0"/>
-      <limit lower="-3.31" upper="3.31" effort="0" velocity="6.98"/>
+      <limit lower="-1.57" upper="1.57" effort="0" velocity="6.98"/>
     </joint>
     <joint name="${prefix}joint_5" type="revolute">

Commit message: Fix axis limits for "integrated J3 cable" M-10iA version

File: fanuc_m10ia_support/urdf/m10ia_macro.xacro (robot description, xacro)
@@ -145,5 +145,5 @@
       <child link="${prefix}link_5"/>
       <axis xyz="0 -1 0"/>
-      <limit lower="-3.31" upper="3.31" effort="0" velocity="6.98"/>
+      <limit lower="-2.41" upper="2.44" effort="0" velocity="6.98"/>
     </joint>
     <joint name="${prefix}joint_6" type="revolute">
@@ -152,5 +152,5 @@
       <child link="${prefix}link_6"/>
       <axis xyz="-1 0 0"/>
-      <limit lower="-6.28" upper="6.28" effort="0" velocity="10.47"/>
+      <limit lower="-4.71" upper="4.71" effort="0" velocity="10.47"/>
     </joint>
     <joint name="${prefix}joint_6-tool0" type="fixed">

Commit message: Change axis 2 limit

File: fanuc_m10ia_support/urdf/m10ia_macro.xacro (robot description, xacro)
@@ -124,5 +124,5 @@
       <child link="${prefix}link_2"/>
       <axis xyz="0 1 0"/>
-      <limit lower="-1.57" upper="2.79" effort="0" velocity="3.32"/>
+      <limit lower="-1.57" upper="1.57" effort="0" velocity="3.32"/>
     </joint>
     <joint name="${prefix}joint_3" type="revolute">
