Commit message: DAE meshes

File: fanuc_m10ia_support/urdf/m10ia.urdf (robot description, URDF)
Before this commit: robot fanuc_m10ia, 9 links, 8 joints
Links:
- link link_1: geometry collision mesh filename=package://fanuc_m10ia_support/meshes/m10ia/collision/link_1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; visual mesh filename=package://fanuc_m10ia_support/meshes/m10ia/visual/link_1.dae
- link link_2: geometry collision mesh filename=package://fanuc_m10ia_support/meshes/m10ia/collision/link_2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; visual mesh filename=package://fanuc_m10ia_support/meshes/m10ia/visual/link_2.dae
- link link_3: geometry collision mesh filename=package://fanuc_m10ia_support/meshes/m10ia/collision/link_3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; visual mesh filename=package://fanuc_m10ia_support/meshes/m10ia/visual/link_3.dae
- link link_4: geometry collision mesh filename=package://fanuc_m10ia_support/meshes/m10ia/collision/link_4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; visual mesh filename=package://fanuc_m10ia_support/meshes/m10ia/visual/link_4.dae
- link link_5: geometry collision mesh filename=package://fanuc_m10ia_support/meshes/m10ia/collision/link_5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; visual mesh filename=package://fanuc_m10ia_support/meshes/m10ia/visual/link_5.dae
- link link_6: geometry collision mesh filename=package://fanuc_m10ia_support/meshes/m10ia/collision/link_6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; visual mesh filename=package://fanuc_m10ia_support/meshes/m10ia/visual/link_6.dae

File: fanuc_m10ia_support/urdf/m10ia_macro.xacro (robot description, xacro)
@@ -9,5 +9,5 @@
         <origin xyz="0 0 0" rpy="0 0 0"/>
         <geometry>
-          <mesh filename="package://fanuc_m10ia_support/meshes/m10ia/visual/base_link.stl"/>
+          <mesh filename="package://fanuc_m10ia_support/meshes/m10ia/visual/base_link.dae"/>
         </geometry>
         <xacro:material_fanuc_grey />
@@ -24,5 +24,5 @@
         <origin xyz="0 0 0" rpy="0 0 0"/>
         <geometry>
-          <mesh filename="package://fanuc_m10ia_support/meshes/m10ia/visual/link_1.stl"/>
+          <mesh filename="package://fanuc_m10ia_support/meshes/m10ia/visual/link_1.dae"/>
         </geometry>
         <xacro:material_fanuc_yellow />
@@ -39,5 +39,5 @@
         <origin xyz="0 0 0" rpy="0 0 0"/>
         <geometry>
-          <mesh filename="package://fanuc_m10ia_support/meshes/m10ia/visual/link_2.stl"/>
+          <mesh filename="package://fanuc_m10ia_support/meshes/m10ia/visual/link_2.dae"/>
         </geometry>
         <xacro:material_fanuc_yellow />
@@ -54,5 +54,5 @@
         <origin xyz="0 0 0" rpy="0 0 0"/>
         <geometry>
-          <mesh filename="package://fanuc_m10ia_support/meshes/m10ia/visual/link_3.stl"/>
+          <mesh filename="package://fanuc_m10ia_support/meshes/m10ia/visual/link_3.dae"/>
         </geometry>
         <xacro:material_fanuc_yellow />
@@ -69,5 +69,5 @@
         <origin xyz="0 0 0" rpy="0 0 0"/>
         <geometry>
-          <mesh filename="package://fanuc_m10ia_support/meshes/m10ia/visual/link_4.stl"/>
+          <mesh filename="package://fanuc_m10ia_support/meshes/m10ia/visual/link_4.dae"/>
         </geometry>
         <xacro:material_fanuc_yellow />
@@ -84,5 +84,5 @@
         <origin xyz="0 0 0" rpy="0 0 0"/>
         <geometry>
-          <mesh filename="package://fanuc_m10ia_support/meshes/m10ia/visual/link_5.stl"/>
+          <mesh filename="package://fanuc_m10ia_support/meshes/m10ia/visual/link_5.dae"/>
         </geometry>
         <xacro:material_fanuc_yellow />
@@ -99,5 +99,5 @@
         <origin xyz="0 0 0" rpy="0 0 0"/>
         <geometry>
-          <mesh filename="package://fanuc_m10ia_support/meshes/m10ia/visual/link_6.stl"/>
+          <mesh filename="package://fanuc_m10ia_support/meshes/m10ia/visual/link_6.dae"/>
         </geometry>
         <xacro:material_fanuc_black />
